File: eagle/808_CB.brd (EAGLE design)
At the start: 100.8 x 81.3 mm, 56 parts, among them IC1 4584N, IC2 TL072P, Q1 2N3904, Q2 2N3904, Q3 2N3904, Q4 2N3906, X1 22-23-2021

Commit message: switch back oscillator caps
Parts:
- R5: value 330K -> 100K
- R6: value 390k -> 150k
Changed lines of the file:
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@@
 <?xml version="1.0" encoding="utf-8"?>
 <!DOCTYPE eagle SYSTEM "eagle.dtd">
-<eagle version="7.2.0">
+<eagle version="7.1.0">
 <drawing>
 <settings>
@@
 <element name="R22" library="TR808clone" package="0207/5V" value="22K" x="45.974" y="49.276"/>
 <element name="R8" library="TR808clone" package="0207/7" value="33k" x="13.335" y="60.452" rot="R270"/>
-<element name="R5" library="TR808clone" package="0207/5V" value="330K" x="13.716" y="66.802"/>
-<element name="R6" library="TR808clone" package="0207/5V" value="390k" x="24.765" y="61.976" rot="R90"/>
+<element name="R5" library="TR808clone" package="0207/5V" value="100K" x="13.716" y="66.802"/>
+<element name="R6" library="TR808clone" package="0207/5V" value="150k" x="24.765" y="61.976" rot="R90"/>
 <element name="R23" library="TR808clone" package="0207/5V" value="10K" x="48.26" y="54.864" rot="R270"/>
 <element name="R9" library="TR808clone" package="0207/5V" value="2k2" x="33.274" y="55.626" rot="R270"/>
