File: eagle/808_CB.sch (EAGLE design)
At the start: 54 parts, among them IC1 4584N, IC4 TL072P, Q1 2N3904, Q2 2N3904, Q3 2N3904, Q8 2N3906

Commit message: part by part
Parts:
- removed 540HZ, 800HZ: 200k, pot:3RP/1610N
- removed R3*: 22K, TR808clone:R-EU_0207/5V
- added R26: 1k, TR808clone:R-EU_0207/5V
- added R27: 8k2, TR808clone:R-EU_0207/5V
- added R29: 22k, TR808clone:R-EU_0207/5V
- C10: value 3.3n -> 0.47uF/50; device TR808clone:C-EU3.5MM_PITCH -> rcl:CPOL-USB45181A
- C5: value 0.47uF/50 -> 2.2n; device rcl:CPOL-USB45181A -> TR808clone:C-EU3.5MM_PITCH
- C6: value 1uF/50 -> 2.2n; device rcl:CPOL-USB45181A -> TR808clone:C-EU3.5MM_PITCH
- C7: value 2.2n -> 3.3n
- C8: value 2.2n -> 10n
- C9: value 10n -> 1uF/50; device TR808clone:C-EU3.5MM_PITCH -> rcl:CPOL-USB45181A
- R10, R9: value 470k -> 2k2
- R11, R12: value 100R -> 470k
- R13: value 1k -> 100R
- R14: value 33k -> 100R
- R20: value 470k -> 33k
- R21: value 8k2 -> 470k
- R22: value 22k -> 22K
- R3, R4: value 33k -> 200k; device TR808clone:R-EU_0207/5V -> pot:3RP/1610N
- R7, R8: value 2k2 -> 33k
- renumbered 540HZ1 to R28, IC4 to IC2, OUTPUT to JCK1, OUT_NORM to X1, Q8 to Q4, R10* to R25, R15* to R24, R166* to R30, R6* to R23
Connections:
- net +15V: now also R11.2, R12.2; no longer R10.2, R9.2
- net GND: now also C10.-, C9.-, R10.1, R13.1, R14.1, R29.1, R9.1; no longer C5.-, C6.-, R11.1, R12.1, R22.1, R7.1, R8.1
- net LT: now also R22.2; no longer R3*.2
- net N$10: now also R9.2; no longer R3.2
- net N$11: now also R12.1; no longer R10.1
- net N$12: now also R11.1; no longer R9.1
- net N$13: now also R13.2; no longer R11.2
- net N$14: now also R14.2; no longer R12.2
- net N$15: now also D2.C; no longer D1.C
- net N$16: now also D1.C; no longer D2.C
- net N$17: now also C10.+, R20.2; no longer C5.+, R14.2
- net N$18: now also R26.2; no longer R13.2
- net N$19: now also R26.1; no longer R13.1
- net N$20: now also C9.+, R20.1; no longer C6.+, R14.1
- net N$21: now also D2.A; no longer D1.A
- net N$22: now also D1.A; no longer D2.A
- net N$23: now also C5.1; no longer C8.1
- net N$24: now also C6.1; no longer C7.1
- net N$25: now also C5.2, C6.2, C7.1, C8.1; no longer C10.1, C7.2, C8.2, C9.1
- net N$26: now also C8.2, R21.1; no longer C9.2, R20.1
- net N$27: now also C7.2, R21.2; no longer C10.2, R20.2
- net N$29: now also R27.1; no longer R21.1
- net N$30: now also R27.2; no longer R21.2
- net N$32: now also R29.2; no longer R22.2
- net N$4: now also R4.S; no longer 800HZ.S
- net N$5: now also R3.S; no longer 540HZ.S
- net N$517: now also R22.1; no longer R3*.1
- net N$6: now also R7.1; no longer R3.1
- net N$7: now also R3.E; no longer 540HZ.E
- net N$8: now also R4.E; no longer 800HZ.E
- net N$9: now also R10.2; no longer R4.2
- net TP7: now also R8.1; no longer R4.1
Other:
- moved on the sheet: C7, C8, D1, D2, R10, R11, R12, R13, R14, R20, R21, R22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

Commit message: parts on the board
Parts:
- renumbered R28 to LEVEL, R3 to TUNE_1, R4 to TUNE_2
Changed lines of the file:
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@@
 <part name="GND3" library="supply1" deviceset="GND" device=""/>
 <part name="P+2" library="supply1" deviceset="+5V" device=""/>
-<part name="R3" library="pot" deviceset="3RP/1610N" device="" value="200k"/>
-<part name="R4" library="pot" deviceset="3RP/1610N" device="" value="200k"/>
+<part name="TUNE_1" library="pot" deviceset="3RP/1610N" device="" value="200k"/>
+<part name="TUNE_2" library="pot" deviceset="3RP/1610N" device="" value="200k"/>
 <part name="R1" library="TR808clone" deviceset="R-EU_" device="0207/5V" value="20K"/>
 <part name="R2" library="TR808clone" deviceset="R-EU_" device="0207/5V" value="20K"/>
@@
 <part name="GND12" library="supply1" deviceset="GND" device=""/>
 <part name="R27" library="TR808clone" deviceset="R-EU_" device="0207/5V" value="8k2"/>
-<part name="R28" library="pot" deviceset="3RP/1610N" device="" value="5kA"/>
+<part name="LEVEL" library="pot" deviceset="3RP/1610N" device="" value="5kA"/>
 <part name="GND15" library="supply1" deviceset="GND" device=""/>
 <part name="C12" library="TR808clone" deviceset="C-EU" device="3.5MM_PITCH" value="22n"/>
@@
 <instance part="GND3" gate="1" x="-25.4" y="30.48"/>
 <instance part="P+2" gate="1" x="-25.4" y="53.34"/>
-<instance part="R3" gate="G$1" x="-33.02" y="50.8" rot="R90"/>
-<instance part="R4" gate="G$1" x="-30.48" y="15.24" rot="R90"/>
+<instance part="TUNE_1" gate="G$1" x="-33.02" y="50.8" rot="R90"/>
+<instance part="TUNE_2" gate="G$1" x="-30.48" y="15.24" rot="R90"/>
 <instance part="R1" gate="G$1" x="-48.26" y="45.72" rot="R90"/>
 <instance part="R2" gate="G$1" x="-48.26" y="10.16" rot="R90"/>
@@
 <attribute name="VALUE" x="144.018" y="-3.81" size="1.778" layer="96" rot="MR90"/>
 </instance>
-<instance part="R28" gate="G$1" x="139.7" y="-15.24"/>
+<instance part="LEVEL" gate="G$1" x="139.7" y="-15.24"/>
 <instance part="GND15" gate="1" x="139.7" y="-33.02"/>
 <instance part="C12" gate="G$1" x="149.86" y="-15.24" rot="R90"/>
@@
 </segment>
 <segment>
-<pinref part="R28" gate="G$1" pin="A"/>
+<pinref part="LEVEL" gate="G$1" pin="A"/>
 <pinref part="GND15" gate="1" pin="GND"/>
 <wire x1="139.7" y1="-30.48" x2="139.7" y2="-20.32" width="0.1524" layer="91"/>
@@
 <pinref part="R5" gate="G$1" pin="1"/>
 <wire x1="-30.48" y1="20.32" x2="-25.4" y2="20.32" width="0.1524" layer="91"/>
-<pinref part="R4" gate="G$1" pin="S"/>
+<pinref part="TUNE_2" gate="G$1" pin="S"/>
 </segment>
 </net>
@@
 <pinref part="R6" gate="G$1" pin="1"/>
 <wire x1="-33.02" y1="55.88" x2="-22.86" y2="55.88" width="0.1524" layer="91"/>
-<pinref part="R3" gate="G$1" pin="S"/>
+<pinref part="TUNE_1" gate="G$1" pin="S"/>
 </segment>
 </net>
@@
 <segment>
 <pinref part="R1" gate="G$1" pin="2"/>
-<pinref part="R3" gate="G$1" pin="E"/>
+<pinref part="TUNE_1" gate="G$1" pin="E"/>
 <wire x1="-48.26" y1="50.8" x2="-38.1" y2="50.8" width="0.1524" layer="91"/>
 </segment>
@@
 <segment>
 <pinref part="R2" gate="G$1" pin="2"/>
-<pinref part="R4" gate="G$1" pin="E"/>
+<pinref part="TUNE_2" gate="G$1" pin="E"/>
 <wire x1="-48.26" y1="15.24" x2="-35.56" y2="15.24" width="0.1524" layer="91"/>
 </segment>
@@
 <segment>
 <pinref part="R27" gate="G$1" pin="1"/>
-<pinref part="R28" gate="G$1" pin="E"/>
+<pinref part="LEVEL" gate="G$1" pin="E"/>
 <wire x1="139.7" y1="-10.16" x2="139.7" y2="-5.08" width="0.1524" layer="91"/>
 </segment>
@@
 <segment>
 <pinref part="C12" gate="G$1" pin="1"/>
-<pinref part="R28" gate="G$1" pin="S"/>
+<pinref part="LEVEL" gate="G$1" pin="S"/>
 <wire x1="147.32" y1="-15.24" x2="144.78" y2="-15.24" width="0.1524" layer="91"/>
 </segment>

Commit message: routed
Parts:
- R8: device TR808clone:R-EU_0207/5V -> TR808clone:R-EU_0207/7
Changed lines of the file:
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@@
 <grid distance="0.1" unitdist="inch" unit="inch" style="lines" multiple="1" display="no" altdistance="0.01" altunitdist="inch" altunit="inch"/>
 <layers>
-<layer number="1" name="Top" color="1" fill="1" visible="no" active="no"/>
-<layer number="16" name="Bottom" color="4" fill="1" visible="no" active="no"/>
-<layer number="17" name="Pads" color="2" fill="1" visible="no" active="no"/>
-<layer number="18" name="Vias" color="2" fill="1" visible="no" active="no"/>
-<layer number="19" name="Unrouted" color="6" fill="1" visible="no" active="no"/>
-<layer number="20" name="Dimension" color="15" fill="1" visible="no" active="no"/>
-<layer number="21" name="tPlace" color="7" fill="1" visible="no" active="no"/>
-<layer number="22" name="bPlace" color="7" fill="1" visible="no" active="no"/>
-<layer number="23" name="tOrigins" color="15" fill="1" visible="no" active="no"/>
-<layer number="24" name="bOrigins" color="15" fill="1" visible="no" active="no"/>
-<layer number="25" name="tNames" color="7" fill="1" visible="no" active="no"/>
-<layer number="26" name="bNames" color="7" fill="1" visible="no" active="no"/>
-<layer number="27" name="tValues" color="7" fill="1" visible="no" active="no"/>
-<layer number="28" name="bValues" color="7" fill="1" visible="no" active="no"/>
-<layer number="29" name="tStop" color="7" fill="6" visible="no" active="no"/>
-<layer number="30" name="bStop" color="7" fill="3" visible="no" active="no"/>
-<layer number="31" name="tCream" color="7" fill="5" visible="no" active="no"/>
-<layer number="32" name="bCream" color="7" fill="4" visible="no" active="no"/>
+<layer number="1" name="Top" color="4" fill="1" visible="yes" active="no"/>
+<layer number="16" name="Bottom" color="1" fill="1" visible="yes" active="no"/>
+<layer number="17" name="Pads" color="2" fill="1" visible="yes" active="no"/>
+<layer number="18" name="Vias" color="2" fill="1" visible="yes" active="no"/>
+<layer number="19" name="Unrouted" color="6" fill="1" visible="yes" active="no"/>
+<layer number="20" name="Dimension" color="15" fill="1" visible="yes" active="no"/>
+<layer number="21" name="tPlace" color="7" fill="1" visible="yes" active="no"/>
+<layer number="22" name="bPlace" color="7" fill="1" visible="yes" active="no"/>
+<layer number="23" name="tOrigins" color="15" fill="1" visible="yes" active="no"/>
+<layer number="24" name="bOrigins" color="15" fill="1" visible="yes" active="no"/>
+<layer number="25" name="tNames" color="7" fill="1" visible="yes" active="no"/>
+<layer number="26" name="bNames" color="7" fill="1" visible="yes" active="no"/>
+<layer number="27" name="tValues" color="7" fill="1" visible="yes" active="no"/>
+<layer number="28" name="bValues" color="7" fill="1" visible="yes" active="no"/>
+<layer number="29" name="tStop" color="7" fill="3" visible="no" active="no"/>
+<layer number="30" name="bStop" color="7" fill="6" visible="no" active="no"/>
+<layer number="31" name="tCream" color="7" fill="4" visible="no" active="no"/>
+<layer number="32" name="bCream" color="7" fill="5" visible="no" active="no"/>
 <layer number="33" name="tFinish" color="6" fill="3" visible="no" active="no"/>
 <layer number="34" name="bFinish" color="6" fill="6" visible="no" active="no"/>
 <layer number="35" name="tGlue" color="7" fill="4" visible="no" active="no"/>
 <layer number="36" name="bGlue" color="7" fill="5" visible="no" active="no"/>
-<layer number="37" name="tTest" color="7" fill="1" visible="no" active="no"/>
-<layer number="38" name="bTest" color="7" fill="1" visible="no" active="no"/>
+<layer number="37" name="tTest" color="7" fill="1" visible="yes" active="no"/>
+<layer number="38" name="bTest" color="7" fill="1" visible="yes" active="no"/>
 <layer number="39" name="tKeepout" color="4" fill="11" visible="no" active="no"/>
 <layer number="40" name="bKeepout" color="1" fill="11" visible="no" active="no"/>
@@
 <layer number="44" name="Drills" color="7" fill="1" visible="no" active="no"/>
 <layer number="45" name="Holes" color="7" fill="1" visible="no" active="no"/>
-<layer number="46" name="Milling" color="3" fill="1" visible="no" active="no"/>
-<layer number="47" name="Measures" color="7" fill="1" visible="no" active="no"/>
-<layer number="48" name="Document" color="7" fill="1" visible="no" active="no"/>
-<layer number="49" name="Reference" color="7" fill="1" visible="no" active="no"/>
-<layer number="50" name="dxf" color="7" fill="1" visible="no" active="no"/>
-<layer number="51" name="tDocu" color="7" fill="1" visible="no" active="no"/>
-<layer number="52" name="bDocu" color="7" fill="1" visible="no" active="no"/>
-<layer number="53" name="tGND_GNDA" color="7" fill="9" visible="no" active="no"/>
-<layer number="54" name="bGND_GNDA" color="1" fill="9" visible="no" active="no"/>
-<layer number="56" name="wert" color="7" fill="1" visible="no" active="no"/>
-<layer number="57" name="tCAD" color="7" fill="1" visible="no" active="no"/>
-<layer number="59" name="tCarbon" color="7" fill="1" visible="no" active="no"/>
-<layer number="60" name="bCarbon" color="7" fill="1" visible="no" active="no"/>
+<layer number="46" name="Milling" color="3" fill="1" visible="yes" active="no"/>
+<layer number="47" name="Measures" color="7" fill="1" visible="yes" active="no"/>
+<layer number="48" name="Document" color="7" fill="1" visible="yes" active="no"/>
+<layer number="49" name="Reference" color="7" fill="1" visible="yes" active="no"/>
+<layer number="50" name="dxf" color="7" fill="1" visible="yes" active="no"/>
+<layer number="51" name="tDocu" color="7" fill="1" visible="yes" active="no"/>
+<layer number="52" name="bDocu" color="7" fill="1" visible="yes" active="no"/>
+<layer number="53" name="tGND_GNDA" color="7" fill="9" visible="yes" active="no"/>
+<layer number="54" name="bGND_GNDA" color="1" fill="9" visible="yes" active="no"/>
+<layer number="56" name="wert" color="7" fill="1" visible="yes" active="no"/>
+<layer number="57" name="tCAD" color="7" fill="1" visible="yes" active="no"/>
+<layer number="59" name="tCarbon" color="7" fill="1" visible="yes" active="no"/>
+<layer number="60" name="bCarbon" color="7" fill="1" visible="yes" active="no"/>
 <layer number="90" name="Modules" color="5" fill="1" visible="yes" active="yes"/>
 <layer number="91" name="Nets" color="2" fill="1" visible="yes" active="yes"/>
@@
 <part name="P+3" library="supply1" deviceset="+5V" device=""/>
 <part name="R7" library="TR808clone" deviceset="R-EU_" device="0207/5V" value="33k"/>
-<part name="R8" library="TR808clone" deviceset="R-EU_" device="0207/5V" value="33k"/>
+<part name="R8" library="TR808clone" deviceset="R-EU_" device="0207/7" value="33k"/>
 <part name="R9" library="TR808clone" deviceset="R-EU_" device="0207/5V" value="2k2"/>
 <part name="GND4" library="supply1" deviceset="GND" device=""/>
